Commit message: solver correction

File: genesis/assets/urdf/lisparrow/lisparrow.urdf (robot description, URDF)
Before this commit: robot lisparrow, 15 links, 14 joints
Joints:
- joint fixed_joint_aero_frame_center_wing: origin xyz=0 0 0 rpy=3.141600 -1.570800 -1.5708 -> xyz=0 0 0 rpy=0.785399 -1.570791 0.785399
- joint fixed_joint_aero_frame_elevator: origin xyz=0 0 0 rpy=0.047733 -1.570807 1.5708 -> xyz=0 0 0 rpy=3.141516 1.523067 1.570720
- joint fixed_joint_aero_frame_left_outer_wing: origin xyz=0 0 0 rpy=2.034429 -1.570788 4.2488 -> xyz=0 0 0 rpy=1.570804 0.000000 -3.141589
- joint fixed_joint_aero_frame_right_outer_wing: origin xyz=0 0 0 rpy=-0.000104 1.570793 0.0072 -> xyz=0 0 0 rpy=-1.570797 0.000000 3.141589
- joint fixed_joint_aero_frame_rudder: origin xyz=0 0 0 rpy=0.000000 -1.570807 1.5708 -> xyz=0 0 0 rpy=0.785399 1.570791 -0.785399

Commit message: 172

File: genesis/assets/urdf/lisparrow/lisparrow.urdf (robot description, URDF)
Before this commit: robot lisparrow, 15 links, 14 joints
Joints:
- joint elevator_pitch_joint: axis 0 0 0 -> 1 0 0
- joint fixed_joint_aero_frame_center_wing: origin xyz=0 0 0 rpy=0.785399 -1.570791 0.785399 -> xyz=0 0 0.045 rpy=0.785399 -1.570791 0.785399
- joint fixed_joint_aero_frame_elevator: origin xyz=0 0 0 rpy=3.141516 1.523067 1.570720 -> xyz=0 0 0.0145 rpy=3.141516 1.523067 1.570720
- joint fixed_joint_aero_frame_left_outer_wing: origin xyz=0 0 0 rpy=1.570804 0.000000 -3.141589 -> xyz=-0.0375 0 0 rpy=1.570804 0.000000 -3.141589
- joint fixed_joint_aero_frame_right_outer_wing: origin xyz=0 0 0 rpy=-1.570797 0.000000 3.141589 -> xyz=-0.0375 0 0 rpy=-1.570797 0.000000 3.141589
- joint fixed_joint_aero_frame_rudder: origin xyz=0 0 0 rpy=0.785399 1.570791 -0.785399 -> xyz=0 0 0.024 rpy=0.785399 1.570791 -0.785399
- joint joint_0_sweep_left_wing: axis 0 0 0 -> 0 -1 0; origin xyz=-0.1385 -0.00035 0.128 rpy=3.1416 1.5708 0 -> xyz=-0.1385 -0.00035 0.0 rpy=3.1416 1.5708 0
- joint joint_0_sweep_right_wing: axis 0 0 0 -> 0 1 0; origin xyz=0.1385 -0.00415 0.128 rpy=0 1.5708 0 -> xyz=0.1385 -0.00035 0.0 rpy=0 1.5708 0
- joint rudder_yaw_joint: axis 0 0 0 -> 0 1 0

File: genesis/assets/urdf/mydrone/[0.7, 3.5, 0.73, 0.38, 0.38, 0.5, 4, 0.2, 2, 0, 2, 2.5, 3, 4, 16].urdf (robot description, URDF)
Before this commit: robot drone_param, 26 links, 25 joints
Links:
- link elevator_hinge: mass 0.01 -> 0.02; geometry visual mesh filename=package://meshes/elevator.stl scale=0.000625262 0.00166667 0.00147528
- link elevator_left: mass 0.00847298 -> 0.0085; geometry collision box size=0.02 0.125 0.25
- link elevator_right: mass 0.00847298 -> 0.0085; geometry collision box size=0.02 0.125 0.25
- link fuselage: mass 0.402961 -> 0.275575
- link fuselage_left_0: mass 0.01 -> 0.005
- link fuselage_left_1: mass 0.01 -> 0.005
- link fuselage_right_0: mass 0.01 -> 0.005
- link fuselage_right_1: mass 0.01 -> 0.005
- link left_wing: mass 0.0502942 -> 0.060928; geometry collision box size=0.032 0.2 0.7; visual mesh filename=package://meshes/wing0009.stl scale=0.200012 0.7 0.356303
- link prop_camera_payload: mass 0.05 -> 0.03
- link right_wing: mass 0.0502942 -> 0.060928; geometry collision box size=0.032 0.2 0.7; visual mesh filename=package://meshes/wing0009.stl scale=0.200012 0.7 0.356303
- link rudder: mass 0.0054227 -> 0.004352; geometry collision box size=0.016 0.1 0.2; visual mesh filename=package://meshes/rudder.stl scale=0.000670449 0.00118022 0.00122269

File: src/urdf_generated/[0.7, 3.5, 0.73, 0.38, 0.38, 0.5, 4, 0.2, 2, -10, 2, 2.5, 3, 4, 16].urdf (robot description, URDF)
Before this commit: robot drone_param, 26 links, 25 joints
Links:
- link elevator_hinge: mass 0.01 -> 0.02; geometry visual mesh filename=package://meshes/elevator.stl scale=0.000625262 0.00166667 0.00147528
- link elevator_left: mass 0.00752992 -> 0.0085; geometry collision box size=0.02 0.125 0.25
- link elevator_right: mass 0.00752992 -> 0.0085; geometry collision box size=0.02 0.125 0.25
- link fuselage: mass 0.377775 -> 0.275575; geometry collision box size=0.1 0.104768037946 0.73; visual mesh filename=package://meshes/fuselage_only.stl scale=0.000973482 0.001 0.001
- link fuselage_left_0: mass 0.01 -> 0.005
- link fuselage_left_1: mass 0.01 -> 0.005
- link fuselage_right_0: mass 0.01 -> 0.005
- link fuselage_right_1: mass 0.01 -> 0.005
- link left_wing: mass 0.0865724 -> 0.060928; geometry collision box size=0.032 0.2 0.7; visual mesh filename=package://meshes/wing0009.stl scale=0.200012 0.7 0.356303
- link prop_camera_payload: mass 0.05 -> 0.03
- link right_wing: mass 0.0865724 -> 0.060928; geometry collision box size=0.032 0.2 0.7; visual mesh filename=package://meshes/wing0009.stl scale=0.200012 0.7 0.356303
- link rudder: mass 0.00210482 -> 0.004352; geometry collision box size=0.016 0.1 0.2; visual mesh filename=package://meshes/rudder.stl scale=0.000670449 0.00118022 0.00122269
Joints:
- joint elevator_pitch_joint: origin xyz=-0.639800576241 0 0 rpy=0 0 0 -> xyz=-0.76 0 0 rpy=0 0 0
- joint fixed_joint_aero_frame_elevator_left: origin xyz=-0.0366623805319 0 0 rpy=0 3.141592654 0 -> xyz=-0.03125 0 0 rpy=0 3.141592654 0
- joint fixed_joint_aero_frame_elevator_right: origin xyz=-0.0366623805319 0 0 rpy=0 3.141592654 0 -> xyz=-0.03125 0 0 rpy=0 3.141592654 0
- joint fixed_joint_aero_frame_fuselage: origin xyz=-0.222732054872 0 -0.03 rpy=0 3.141592653589793 0 -> xyz=-0.2774 0 -0.03 rpy=0 3.141592653589793 0
- joint fixed_joint_aero_frame_left_wing: origin xyz=0 0.359844163834 0 rpy=0 3.141592654 0 -> xyz=0 0.35 0 rpy=0 3.141592654 0
- joint fixed_joint_aero_frame_right_wing: origin xyz=0 -0.359844163834 0 rpy=0 3.141592654 0 -> xyz=0 -0.35 0 rpy=0 3.141592654 0
- joint fixed_joint_aero_frame_rudder: origin xyz=-0.0113183289932 0 -0.08 rpy=0 3.141592653589793 0 -> xyz=-0.025 0 -0.08 rpy=0 3.141592653589793 0
- joint fixed_joint_elevator_left: origin xyz=0 0.189375392789 0 rpy=0 0 0 -> xyz=0 0.25 0 rpy=0 0 0
- joint fixed_joint_elevator_right: origin xyz=0 -0.189375392789 0 rpy=0 0 0 -> xyz=0 -0.25 0 rpy=0 0 0
- joint fixed_joint_elevator_servo: origin xyz=-0.639800576241 0 0 rpy=0 0 0 -> xyz=-0.76 0 0 rpy=0 0 0
- joint fixed_joint_left_wing: origin xyz=-0.221545739958 -0.05 -0.03 rpy=-0 0 0 -> xyz=-0.2774 -0.05 -0.03 rpy=0.174532925199 0 0
- joint fixed_joint_right_wing: origin xyz=-0.221545739958 0.05 -0.03 rpy=0 0 0 -> xyz=-0.2774 0.05 -0.03 rpy=-0.174532925199 0 0
- joint joint_0_sweep_left_wing: limit lower=-0.236879 upper=0.236879 effort=2.21632 velocity=3.665191429 -> lower=-0.35 upper=0.35 effort=1.5 velocity=3.665191429
- joint joint_0_sweep_right_wing: limit lower=-0.236879 upper=0.236879 effort=2.21632 velocity=3.665191429 -> lower=-0.35 upper=0.35 effort=1.5 velocity=3.665191429
- joint joint_1_twist_left_wing: limit lower=-0.240405 upper=0.240405 effort=1.2479 velocity=3.665191429 -> lower=-0.2 upper=0.2 effort=1.5 velocity=3.665191429
- joint joint_1_twist_right_wing: limit lower=-0.240405 upper=0.240405 effort=1.2479 velocity=3.665191429 -> lower=-0.2 upper=0.2 effort=1.5 velocity=3.665191429

File: src/urdf_generated/[0.7, 3.5, 0.73, 0.38, 0.38, 0.5, 4, 0.2, 2, 10, 2, 2.5, 3, 4, 16].urdf (robot description, URDF)
Before this commit: robot drone_param, 26 links, 25 joints
Links:
- link elevator_hinge: geometry visual mesh filename=package://meshes/elevator.stl scale=0.000625262 0.00166667 0.001
- link elevator_left: mass 0.00460796 -> 0.00847298; geometry collision box size=0.0135567616 0.125 0.25
- link elevator_right: mass 0.00460796 -> 0.00847298; geometry collision box size=0.0135567616 0.125 0.25
- link fuselage: mass 0.385549 -> 0.402961; geometry collision box size=0.1 0.104768037946 0.73; visual mesh filename=package://meshes/fuselage_only.stl scale=0.000973482 0.001 0.001
- link left_wing: mass 0.0471732 -> 0.0502942; geometry collision box size=0.017962225 0.2 0.7; visual mesh filename=package://meshes/wing0009.stl scale=0.2 0.7 0.200012
- link right_wing: mass 0.0471732 -> 0.0502942; geometry collision box size=0.017962225 0.2 0.7; visual mesh filename=package://meshes/wing0009.stl scale=0.2 0.7 0.200012
- link rudder: mass 0.00107562 -> 0.0054227; geometry collision box size=0.0135567616 0.1 0.2; visual mesh filename=package://meshes/rudder.stl scale=0.000670449 0.001 0.00122269
Joints:
- joint elevator_pitch_joint: origin xyz=-0.67689887684 0 0 rpy=0 0 0 -> xyz=-0.76 0 0 rpy=0 0 0
- joint fixed_joint_aero_frame_elevator_left: origin xyz=-0.0244540270119 0 0 rpy=0 3.141592654 0 -> xyz=-0.03125 0 0 rpy=0 3.141592654 0
- joint fixed_joint_aero_frame_elevator_right: origin xyz=-0.0244540270119 0 0 rpy=0 3.141592654 0 -> xyz=-0.03125 0 0 rpy=0 3.141592654 0
- joint fixed_joint_aero_frame_fuselage: origin xyz=-0.211947742257 0 -0.03 rpy=0 3.141592653589793 0 -> xyz=-0.2774 0 -0.03 rpy=0 3.141592653589793 0
- joint fixed_joint_aero_frame_left_wing: origin xyz=0 0.248845437547 0 rpy=0 3.141592654 0 -> xyz=0 0.35 0 rpy=0 3.141592654 0
- joint fixed_joint_aero_frame_right_wing: origin xyz=0 -0.248845437547 0 rpy=0 3.141592654 0 -> xyz=0 -0.35 0 rpy=0 3.141592654 0
- joint fixed_joint_aero_frame_rudder: origin xyz=-0.00830492562934 0 -0.08 rpy=0 3.141592653589793 0 -> xyz=-0.025 0 -0.08 rpy=0 3.141592653589793 0
- joint fixed_joint_elevator_left: origin xyz=0 0.173745034132 0 rpy=0 0 0 -> xyz=0 0.25 0 rpy=0 0 0
- joint fixed_joint_elevator_right: origin xyz=0 -0.173745034132 0 rpy=0 0 0 -> xyz=0 -0.25 0 rpy=0 0 0
- joint fixed_joint_elevator_servo: origin xyz=-0.67689887684 0 0 rpy=0 0 0 -> xyz=-0.76 0 0 rpy=0 0 0
- joint fixed_joint_left_wing: origin xyz=-0.219503444847 -0.05 -0.03 rpy=-0 0 0 -> xyz=-0.2774 -0.05 -0.03 rpy=-0.174532925199 0 0
- joint fixed_joint_right_wing: origin xyz=-0.219503444847 0.05 -0.03 rpy=0 0 0 -> xyz=-0.2774 0.05 -0.03 rpy=0.174532925199 0 0
- joint joint_0_sweep_left_wing: limit lower=-0.202727 upper=0.202727 effort=2.58969 velocity=3.665191429 -> lower=-0.35 upper=0.35 effort=1.5 velocity=3.665191429
- joint joint_0_sweep_right_wing: limit lower=-0.202727 upper=0.202727 effort=2.58969 velocity=3.665191429 -> lower=-0.35 upper=0.35 effort=1.5 velocity=3.665191429
- joint joint_1_twist_left_wing: limit lower=-0.205145 upper=0.205145 effort=1.46238 velocity=3.665191429 -> lower=-0.2 upper=0.2 effort=1.5 velocity=3.665191429
- joint joint_1_twist_right_wing: limit lower=-0.205145 upper=0.205145 effort=1.46238 velocity=3.665191429 -> lower=-0.2 upper=0.2 effort=1.5 velocity=3.665191429

Commit message: lisparrow

File: genesis/assets/urdf/lisparrow/lisparrow.urdf (robot description, URDF)
Before this commit: robot lisparrow, 15 links, 14 joints
Links:
- removed link aero_frame_center_wing
- removed link aero_frame_elevator
- removed link aero_frame_left_outer_wing
- removed link aero_frame_right_outer_wing
- removed link aero_frame_rudder
- removed link center_wing
- removed link elevator
- removed link horizontal_tail
- removed link left_outer_wing
- removed link propeller
- removed link right_outer_wing
- removed link root_link
- removed link rudder
- removed link vertical_tail
- added link elevator_hinged, mass 0.0031868; collision mesh filename=package://meshes/elevator_hinged.STL; visual mesh filename=package://meshes/elevator_hinged.STL
- added link horizontal_tail_fixed, mass 0.0021828; collision mesh filename=package://meshes/horizontal_tail_fixed.STL; visual mesh filename=package://meshes/horizontal_tail_fixed.STL
- added link left_outer_wing_hinged, mass 0.0055726; collision mesh filename=package://meshes/left_outer_wing_hinged.STL; visual mesh filename=package://meshes/left_outer_wing_hinged.STL
- added link propeller_fixed, mass 0.0028325; collision mesh filename=package://meshes/propeller_fixed.STL; visual mesh filename=package://meshes/propeller_fixed.STL
- added link right_outer_wing_hinged, mass 0.0055726; collision mesh filename=package://meshes/right_outer_wing_hinged.STL; visual mesh filename=package://meshes/right_outer_wing_hinged.STL
- added link root_wing_fixed, mass 0.036045; collision mesh filename=package://meshes/root_wing_fixed.STL; visual mesh filename=package://meshes/root_wing_fixed.STL
- added link rudder_hinged, mass 0.0025864; collision mesh filename=package://meshes/rudder_hinged.STL; visual mesh filename=package://meshes/rudder_hinged.STL
- added link vertical_tail_fixed, mass 0.0011935; collision mesh filename=package://meshes/vertical_tail_fixed.STL; visual mesh filename=package://meshes/vertical_tail_fixed.STL
- link fuselage: mass 0.06883 -> 0.064126; geometry collision mesh filename=package://meshes/fuselage.STL; visual mesh filename=package://meshes/fuselage.STL
Joints:
- removed joint elevator_pitch_joint
- removed joint fixed_joint_aero_frame_center_wing
- removed joint fixed_joint_aero_frame_elevator
- removed joint fixed_joint_aero_frame_left_outer_wing
- removed joint fixed_joint_aero_frame_right_outer_wing
- removed joint fixed_joint_aero_frame_rudder
- removed joint fixed_joint_base_fuselage
- removed joint fixed_joint_center_wing
- removed joint fixed_joint_horizontal_tail
- removed joint fixed_joint_propeller
- removed joint fixed_joint_vertical_tail
- removed joint joint_0_sweep_left_wing
- removed joint joint_0_sweep_right_wing
- removed joint rudder_yaw_joint
- added joint joint_elevator_hinged: type revolute, parent horizontal_tail_fixed, child elevator_hinged, origin xyz=-0.39899772195773 0 -0.000545430496194116 rpy=0 0 0, axis 0 -1 0, limit lower=-0.5 upper=0.5 effort=1.0 velocity=3.665191429
- added joint joint_horizontal_tail_fixed: type fixed, parent fuselage, child horizontal_tail_fixed, origin xyz=0 0 0 rpy=0 0 0, axis 0 0 0
- added joint joint_left_outer_wing_hinged: type revolute, parent root_wing_fixed, child left_outer_wing_hinged, origin xyz=-0.0144999999999965 0.1735 0 rpy=0 0 0, axis 0 0 -1, limit lower=-1.4 upper=0.2 effort=1.5 velocity=3.665191429
- added joint joint_propeller_fixed: type fixed, parent fuselage, child propeller_fixed, origin xyz=0 0 0 rpy=0 0 0, axis 0 0 0
- added joint joint_right_outer_wing_hinged: type revolute, parent root_wing_fixed, child right_outer_wing_hinged, origin xyz=-0.0145000000000005 -0.173499999999995 0 rpy=0 0 0, axis 0 0 1, limit lower=-1.4 upper=0.2 effort=1.5 velocity=3.665191429
- added joint joint_root_wing_fixed: type fixed, parent fuselage, child root_wing_fixed, origin xyz=0 0 0 rpy=0 0 0, axis 0 0 0
- added joint joint_rudder_hinged: type revolute, parent vertical_tail_fixed, child rudder_hinged, origin xyz=-0.402 -0.0019749999999986 0.0635500000000013 rpy=0 0 0, axis 0 0 -1, limit lower=-0.5 upper=0.5 effort=1.0 velocity=3.665191429
- added joint joint_vertical_tail_fixed: type fixed, parent fuselage, child vertical_tail_fixed, origin xyz=0 0 0 rpy=0 0 0, axis 0 0 0

Commit message: lisparrow 2

File: genesis/assets/urdf/lisparrow/lisparrow.urdf (robot description, URDF)
Before this commit: robot CAD_Prototype_1_flipped_root_URDF_meshed, 9 links, 8 joints
Joints:
- joint joint_elevator_hinged: limit lower=-0.5 upper=0.5 effort=1.0 velocity=3.665191429 -> lower=-0.5 upper=0.5 effort=1.5 velocity=25.0
- joint joint_left_outer_wing_hinged: limit lower=-1.4 upper=0.2 effort=1.5 velocity=3.665191429 -> lower=-1.4 upper=0.2 effort=1.5 velocity=20.0
- joint joint_right_outer_wing_hinged: limit lower=-1.4 upper=0.2 effort=1.5 velocity=3.665191429 -> lower=-1.4 upper=0.2 effort=1.5 velocity=20.0
- joint joint_rudder_hinged: limit lower=-0.5 upper=0.5 effort=1.0 velocity=3.665191429 -> lower=-0.5 upper=0.5 effort=1.5 velocity=25.0
